Commit message: updated

File: model/robot.xacro (robot description, xacro)
@@ -1,175 +1,188 @@
 <?xml version="1.0"?>
 <robot name="prime" xmlns:xacro="http://www.ros.org/wiki/xacro">
-<xacro:property name="wheel_radius" value="0.1"/>
-<xacro:property name="wheel_thickness" value="0.1"/>
-<xacro:property name="chassis_length" value="0.6"/>
-<xacro:property name="chassis_width" value="0.3"/>
-<xacro:property name="wheel_offset_y" value="${(chassis_width/2)+(wheel_thickness/2)}"/>
-<xacro:property name="chassis_mass" value="0.2"/>
-<xacro:property name="wheel_mass" value="0.02"/>
-<material name="orange">
-<color rgba="1 0.3 0.1 1"/>
-</material>
-<link name="chassis">
-<visual>
-<origin xyz="0 0 0" rpy="0 0 0"/>
-<geometry>
-<box size="${chassis_length} ${chassis_width} 0.1"/>
-</geometry>
-<material name="orange"/>
-</visual>
-<collision>
-<geometry>
-<box size="${chassis_length} ${chassis_width} 0.1"/>
-</geometry>
-<gazebo>
-<mu1>0.8</mu1>
-<mu2>0.2</mu2>
-</gazebo>
-</collision>
-<inertial>
-<mass value="${chassis_mass}"/>
-<inertia ixx="1.0" ixy="0.0" iyy="1.0" izz="1.0" iyz="0.0" ixz="0.0"/>
-</inertial>
-</link>
-<link name="wheel_1">
-<visual>
-<origin xyz="0 0 0" rpy="0 0 0"/>
-<geometry>
-<cylinder radius="${wheel_radius}" length="${wheel_thickness}"/>
-</geometry>
-<material name="orange"/>
-</visual>
-<collision>
-<geometry>
-<cylinder radius="${wheel_radius}" length="${wheel_thickness}"/>
-</geometry>
-<gazebo>
-<mu1>0.8</mu1>
-<mu2>0.2</mu2>
-</gazebo>
-</collision>
-<inertial>
-<mass value="${wheel_mass}"/>
-<inertia ixx="0.1" ixy="0.0" iyy="0.1" iyz="0.0" izz="0.1" ixz="0.0"/>
-</inertial>
-</link>
-<link name="wheel_2">
-<visual>
-<origin xyz="0 0 0" rpy="0 0 0"/>
-<geometry>
-<cylinder radius="${wheel_radius}" length="${wheel_thickness}"/>
-</geometry>
-</visual>
-<collision>
-<geometry>
-<cylinder radius="${wheel_radius}" length="${wheel_thickness}"/>
-</geometry>
-<gazebo>
-<mu1>0.8</mu1>
-<mu2>0.2</mu2>
-</gazebo>
-</collision>
-<inertial>
-<mass value="${wheel_mass}"/>
-<inertia ixx="0.1" ixy="0.0" iyy="0.1" iyz="0.0" izz="0.1" ixz="0.0"/>
-</inertial>
-</link>
-<link name="wheel_3">
-<visual>
-<origin xyz="0 0 0" rpy="0 0 0"/>
-<geometry>
-<cylinder radius="${wheel_radius}" length="${wheel_thickness}"/>
-</geometry>
-</visual>
-<collision>
-<geometry>
-<cylinder radius="${wheel_radius}" length="${wheel_thickness}"/>
-</geometry>
-<gazebo>
-<mu1>0.8</mu1>
-<mu2>0.2</mu2>
-</gazebo>
-</collision>
-<inertial>
-<mass value="${wheel_mass}"/>
-<inertia ixx="0.1" ixy="0.0" iyy="0.1" iyz="0.0" izz="0.1" ixz="0.0"/>
-</inertial>
-</link>
-<link name="wheel_4">
-<visual>
-<origin xyz="0 0 0" rpy="0 0 0"/>
-<geometry>
-<cylinder radius="${wheel_radius}" length="${wheel_thickness}"/>
-</geometry>
-</visual>
-<collision>
-<geometry>
-<cylinder radius="${wheel_radius}" length="${wheel_thickness}"/>
-</geometry>
-</collision>
-<inertial>
-<mass value="${wheel_mass}"/>
-<inertia ixx="0.1" ixy="0.0" iyy="0.1" iyz="0.0" izz="0.1" ixz="0.0"/>
-</inertial>
-</link>
-<joint name="first_wheel_joint" type="revolute">
-<origin xyz="${chassis_length/2} ${-wheel_offset_y} 0" rpy="1.57 0 0"/>
-<parent link="chassis"/>
-<child link="wheel_1"/>
-<limit lower="-3.14" upper="3.14" effort="10" velocity="10"/>
-<axis xyz="0 0 1"/>
-</joint>
-<joint name="second_wheel_joint" type="revolute">
-<origin xyz="${chassis_length/2} ${wheel_offset_y} 0" rpy="1.57 0 0"/>
-<parent link="chassis"/>
-<child link="wheel_2"/>
-<limit lower="-3.14" upper="3.14" effort="10" velocity="10"/>
-<axis xyz="0 0 1"/>
-</joint>
-<joint name="third_wheel_joint" type="revolute">
-<origin xyz="${-chassis_length/2} ${wheel_offset_y} 0" rpy="1.57 0 0"/>
-<parent link="chassis"/>
-<child link="wheel_3"/>
-<limit lower="-3.14" upper="3.14" effort="10" velocity="10"/>
-<axis xyz="0 0 1"/>
-</joint>
-<joint name="fourth_wheel_joint" type="revolute">
-<origin xyz="${-chassis_length/2} ${-wheel_offset_y} 0" rpy="1.57 0 0"/>
-<parent link="chassis"/>
-<child link="wheel_4"/>
-<limit lower="-3.14" upper="3.14" effort="10" velocity="10"/>
-<axis xyz="0 0 1"/>
-</joint>
-<ros2_control name="Gazebosim" type="system">
-<hardware>
-<plugin>gazebo_ros2_control/GazeboSystem</plugin>
-</hardware>
-<joint name="first_wheel_joint">
-<command_interface name="position"/>
-<state_interface name="position"/>
-<state_interface name="velocity"/>
-</joint>
-<joint name="second_wheel_joint">
-<command_interface name="position"/>
-<state_interface name="position"/>
-<state_interface name="velocity"/>
-</joint>
-<joint name="third_wheel_joint">
-<command_interface name="position"/>
-<state_interface name="position"/>
-<state_interface name="velocity"/>
-</joint>
-<joint name="fourth_wheel_joint">
-<command_interface name="position"/>
-<state_interface name="position"/>
-<state_interface name="velocity"/>
-</joint>
-</ros2_control>
-<gazebo>
-<plugin name="gazebo_ros2_control" filename="libgazebo_ros2_control.so">
-  <robotNamespace>/</robotNamespace>
-  <parameters>$(find four_wheel_mobile_robot_navigation)/config/my_controllers.yaml</parameters>
-</plugin>
-</gazebo>
+  <!-- Define new materials -->
+  <material name="red">
+    <color rgba="1 0 0 1"/>
+  </material>
+  <material name="blue">
+    <color rgba="0 0 1 1"/>
+  </material>
+  <!-- Properties -->
+  <xacro:property name="wheel_radius" value="0.1"/>
+  <xacro:property name="wheel_thickness" value="0.1"/>
+  <xacro:property name="chassis_length" value="0.6"/>
+  <xacro:property name="chassis_width" value="0.3"/>
+  <xacro:property name="wheel_offset_y" value="${(chassis_width/2)+(wheel_thickness/2)}"/>
+  <xacro:property name="chassis_mass" value="0.2"/>
+  <xacro:property name="wheel_mass" value="0.02"/>
+  <!-- Chassis link (base) using blue material -->
+  <link name="chassis">
+    <visual>
+      <origin xyz="0 0 0" rpy="0 0 0"/>
+      <geometry>
+        <box size="${chassis_length} ${chassis_width} 0.1"/>
+      </geometry>
+      <material name="blue"/>
+    </visual>
+    <collision>
+      <geometry>
+        <box size="${chassis_length} ${chassis_width} 0.1"/>
+      </geometry>
+      <gazebo>
+        <mu1>0.8</mu1>
+        <mu2>0.2</mu2>
+      </gazebo>
+    </collision>
+    <inertial>
+      <mass value="${chassis_mass}"/>
+      <inertia ixx="1.0" ixy="0.0" iyy="1.0" izz="1.0" iyz="0.0" ixz="0.0"/>
+    </inertial>
+  </link>
+  <!-- Wheel links (all wheels use red material) -->
+  <link name="wheel_1">
+    <visual>
+      <origin xyz="0 0 0" rpy="0 0 0"/>
+      <geometry>
+        <cylinder radius="${wheel_radius}" length="${wheel_thickness}"/>
+      </geometry>
+      <material name="red"/>
+    </visual>
+    <collision>
+      <geometry>
+        <cylinder radius="${wheel_radius}" length="${wheel_thickness}"/>
+      </geometry>
+      <gazebo>
+        <mu1>0.8</mu1>
+        <mu2>0.2</mu2>
+      </gazebo>
+    </collision>
+    <inertial>
+      <mass value="${wheel_mass}"/>
+      <inertia ixx="0.1" ixy="0.0" iyy="0.1" iyz="0.0" izz="0.1" ixz="0.0"/>
+    </inertial>
+  </link>
+  <link name="wheel_2">
+    <visual>
+      <origin xyz="0 0 0" rpy="0 0 0"/>
+      <geometry>
+        <cylinder radius="${wheel_radius}" length="${wheel_thickness}"/>
+      </geometry>
+      <material name="red"/>
+    </visual>
+    <collision>
+      <geometry>
+        <cylinder radius="${wheel_radius}" length="${wheel_thickness}"/>
+      </geometry>
+      <gazebo>
+        <mu1>0.8</mu1>
+        <mu2>0.2</mu2>
+      </gazebo>
+    </collision>
+    <inertial>
+      <mass value="${wheel_mass}"/>
+      <inertia ixx="0.1" ixy="0.0" iyy="0.1" iyz="0.0" izz="0.1" ixz="0.0"/>
+    </inertial>
+  </link>
+  <link name="wheel_3">
+    <visual>
+      <origin xyz="0 0 0" rpy="0 0 0"/>
+      <geometry>
+        <cylinder radius="${wheel_radius}" length="${wheel_thickness}"/>
+      </geometry>
+      <material name="red"/>
+    </visual>
+    <collision>
+      <geometry>
+        <cylinder radius="${wheel_radius}" length="${wheel_thickness}"/>
+      </geometry>
+      <gazebo>
+        <mu1>0.8</mu1>
+        <mu2>0.2</mu2>
+      </gazebo>
+    </collision>
+    <inertial>
+      <mass value="${wheel_mass}"/>
+      <inertia ixx="0.1" ixy="0.0" iyy="0.1" iyz="0.0" izz="0.1" ixz="0.0"/>
+    </inertial>
+  </link>
+  <link name="wheel_4">
+    <visual>
+      <origin xyz="0 0 0" rpy="0 0 0"/>
+      <geometry>
+        <cylinder radius="${wheel_radius}" length="${wheel_thickness}"/>
+      </geometry>
+      <material name="red"/>
+    </visual>
+    <collision>
+      <geometry>
+        <cylinder radius="${wheel_radius}" length="${wheel_thickness}"/>
+      </geometry>
+    </collision>
+    <inertial>
+      <mass value="${wheel_mass}"/>
+      <inertia ixx="0.1" ixy="0.0" iyy="0.1" iyz="0.0" izz="0.1" ixz="0.0"/>
+    </inertial>
+  </link>
+  <!-- Joints -->
+  <joint name="first_wheel_joint" type="revolute">
+    <origin xyz="${chassis_length/2} ${-wheel_offset_y} 0" rpy="1.57 0 0"/>
+    <parent link="chassis"/>
+    <child link="wheel_1"/>
+    <limit lower="-3.14" upper="3.14" effort="10" velocity="10"/>
+    <axis xyz="0 0 1"/>
+  </joint>
+  <joint name="second_wheel_joint" type="revolute">
+    <origin xyz="${chassis_length/2} ${wheel_offset_y} 0" rpy="1.57 0 0"/>
+    <parent link="chassis"/>
+    <child link="wheel_2"/>
+    <limit lower="-3.14" upper="3.14" effort="10" velocity="10"/>
+    <axis xyz="0 0 1"/>
+  </joint>
+  <joint name="third_wheel_joint" type="revolute">
+    <origin xyz="${-chassis_length/2} ${wheel_offset_y} 0" rpy="1.57 0 0"/>
+    <parent link="chassis"/>
+    <child link="wheel_3"/>
+    <limit lower="-3.14" upper="3.14" effort="10" velocity="10"/>
+    <axis xyz="0 0 1"/>
+  </joint>
+  <joint name="fourth_wheel_joint" type="revolute">
+    <origin xyz="${-chassis_length/2} ${-wheel_offset_y} 0" rpy="1.57 0 0"/>
+    <parent link="chassis"/>
+    <child link="wheel_4"/>
+    <limit lower="-3.14" upper="3.14" effort="10" velocity="10"/>
+    <axis xyz="0 0 1"/>
+  </joint>
+  <!-- ros2_control configuration -->
+  <ros2_control name="Gazebosim" type="system">
+    <hardware>
+      <plugin>gazebo_ros2_control/GazeboSystem</plugin>
+    </hardware>
+    <joint name="first_wheel_joint">
+      <command_interface name="position"/>
+      <state_interface name="position"/>
+      <state_interface name="velocity"/>
+    </joint>
+    <joint name="second_wheel_joint">
+      <command_interface name="position"/>
+      <state_interface name="position"/>
+      <state_interface name="velocity"/>
+    </joint>
+    <joint name="third_wheel_joint">
+      <command_interface name="position"/>
+      <state_interface name="position"/>
+      <state_interface name="velocity"/>
+    </joint>
+    <joint name="fourth_wheel_joint">
+      <command_interface name="position"/>
+      <state_interface name="position"/>
+      <state_interface name="velocity"/>
+    </joint>
+  </ros2_control>
+  <!-- Gazebo plugin -->
+  <gazebo>
+    <plugin name="gazebo_ros2_control" filename="libgazebo_ros2_control.so">
+      <robotNamespace>/</robotNamespace>
+      <parameters>$(find four_wheel_mobile_robot_navigation)/config/my_controllers.yaml</parameters>
+    </plugin>
+  </gazebo>
 </robot>

Commit message: updated

File: model/robot.xacro (robot description, xacro)
@@ -1,5 +1,5 @@
 <?xml version="1.0"?>
 <robot name="prime" xmlns:xacro="http://www.ros.org/wiki/xacro">
-  <!-- Define new materials -->
+  <!-- Define materials -->
   <material name="red">
     <color rgba="1 0 0 1"/>
@@ -8,13 +8,21 @@
     <color rgba="0 0 1 1"/>
   </material>
-  <!-- Properties -->
+  <!-- Geometry and mass properties -->
   <xacro:property name="wheel_radius" value="0.1"/>
   <xacro:property name="wheel_thickness" value="0.1"/>
   <xacro:property name="chassis_length" value="0.6"/>
   <xacro:property name="chassis_width" value="0.3"/>
-  <xacro:property name="wheel_offset_y" value="${(chassis_width/2)+(wheel_thickness/2)}"/>
-  <xacro:property name="chassis_mass" value="0.2"/>
-  <xacro:property name="wheel_mass" value="0.02"/>
-  <!-- Chassis link (base) using blue material -->
+  <xacro:property name="wheel_offset_y" value="${(chassis_width/2) + (wheel_thickness/2)}"/>
+  <xacro:property name="chassis_mass" value="5"/>
+  <xacro:property name="wheel_mass" value="0.5"/>
+  <!-- Inertia calculations for the chassis (box shape) -->
+  <xacro:property name="chassis_Ixx" value="${chassis_mass/12 * ((chassis_width**2) + (0.1**2))}"/>
+  <xacro:property name="chassis_Iyy" value="${chassis_mass/12 * ((chassis_length**2) + (0.1**2))}"/>
+  <xacro:property name="chassis_Izz" value="${chassis_mass/12 * ((chassis_length**2) + (chassis_width**2))}"/>
+  <!-- Inertia calculations for the wheels (cylinder shape) -->
+  <xacro:property name="wheel_Ixx" value="${wheel_mass/12 * (3*(wheel_radius**2) + (wheel_thickness**2))}"/>
+  <xacro:property name="wheel_Iyy" value="${wheel_mass/12 * (3*(wheel_radius**2) + (wheel_thickness**2))}"/>
+  <xacro:property name="wheel_Izz" value="${wheel_mass/2 * (wheel_radius**2)}"/>
+  <!-- Chassis Link -->
   <link name="chassis">
     <visual>
@@ -26,18 +34,22 @@
     </visual>
     <collision>
+      <origin xyz="0 0 0" rpy="0 0 0"/>
       <geometry>
         <box size="${chassis_length} ${chassis_width} 0.1"/>
       </geometry>
-      <gazebo>
-        <mu1>0.8</mu1>
-        <mu2>0.2</mu2>
-      </gazebo>
-    </collision>
-    <inertial>
+    </collision>
+    <inertial>
+      <origin xyz="0 0 -0.03"/>
       <mass value="${chassis_mass}"/>
-      <inertia ixx="1.0" ixy="0.0" iyy="1.0" izz="1.0" iyz="0.0" ixz="0.0"/>
-    </inertial>
-  </link>
-  <!-- Wheel links (all wheels use red material) -->
+      <inertia
+          ixx="${chassis_Ixx}"
+          ixy="0.0"
+          iyy="${chassis_Iyy}"
+          izz="${chassis_Izz}"
+          iyz="0.0"
+          ixz="0.0"/>
+    </inertial>
+  </link>
+  <!-- Wheel Links -->
   <link name="wheel_1">
     <visual>
@@ -49,15 +61,24 @@
     </visual>
     <collision>
-      <geometry>
-        <cylinder radius="${wheel_radius}" length="${wheel_thickness}"/>
-      </geometry>
-      <gazebo>
-        <mu1>0.8</mu1>
-        <mu2>0.2</mu2>
-      </gazebo>
-    </collision>
-    <inertial>
-      <mass value="${wheel_mass}"/>
-      <inertia ixx="0.1" ixy="0.0" iyy="0.1" iyz="0.0" izz="0.1" ixz="0.0"/>
+      <origin xyz="0 0 0" rpy="0 0 0"/>
+      <geometry>
+        <cylinder radius="${wheel_radius}" length="${wheel_thickness}"/>
+      </geometry>
+      <gazebo>
+        <mu1>0.6</mu1>
+        <mu2>0.55</mu2>
+        <kp>100000</kp>
+        <kd>500</kd>
+      </gazebo>
+    </collision>
+    <inertial>
+      <mass value="${wheel_mass}"/>
+      <inertia
+          ixx="${wheel_Ixx}"
+          ixy="0.0"
+          iyy="${wheel_Iyy}"
+          izz="${wheel_Izz}"
+          iyz="0.0"
+          ixz="0.0"/>
     </inertial>
   </link>
@@ -71,15 +92,24 @@
     </visual>
     <collision>
-      <geometry>
-        <cylinder radius="${wheel_radius}" length="${wheel_thickness}"/>
-      </geometry>
-      <gazebo>
-        <mu1>0.8</mu1>
-        <mu2>0.2</mu2>
-      </gazebo>
-    </collision>
-    <inertial>
-      <mass value="${wheel_mass}"/>
-      <inertia ixx="0.1" ixy="0.0" iyy="0.1" iyz="0.0" izz="0.1" ixz="0.0"/>
+      <origin xyz="0 0 0" rpy="0 0 0"/>
+      <geometry>
+        <cylinder radius="${wheel_radius}" length="${wheel_thickness}"/>
+      </geometry>
+      <gazebo>
+        <mu1>0.6</mu1>
+        <mu2>0.55</mu2>
+        <kp>100000</kp>
+        <kd>500</kd>
+      </gazebo>
+    </collision>
+    <inertial>
+      <mass value="${wheel_mass}"/>
+      <inertia
+          ixx="${wheel_Ixx}"
+          ixy="0.0"
+          iyy="${wheel_Iyy}"
+          izz="${wheel_Izz}"
+          iyz="0.0"
+          ixz="0.0"/>
     </inertial>
   </link>
@@ -93,15 +123,24 @@
     </visual>
     <collision>
-      <geometry>
-        <cylinder radius="${wheel_radius}" length="${wheel_thickness}"/>
-      </geometry>
-      <gazebo>
-        <mu1>0.8</mu1>
-        <mu2>0.2</mu2>
-      </gazebo>
-    </collision>
-    <inertial>
-      <mass value="${wheel_mass}"/>
-      <inertia ixx="0.1" ixy="0.0" iyy="0.1" iyz="0.0" izz="0.1" ixz="0.0"/>
+      <origin xyz="0 0 0" rpy="0 0 0"/>
+      <geometry>
+        <cylinder radius="${wheel_radius}" length="${wheel_thickness}"/>
+      </geometry>
+      <gazebo>
+        <mu1>0.6</mu1>
+        <mu2>0.55</mu2>
+        <kp>100000</kp>
+        <kd>500</kd>
+      </gazebo>
+    </collision>
+    <inertial>
+      <mass value="${wheel_mass}"/>
+      <inertia
+          ixx="${wheel_Ixx}"
+          ixy="0.0"
+          iyy="${wheel_Iyy}"
+          izz="${wheel_Izz}"
+          iyz="0.0"
+          ixz="0.0"/>
     </inertial>
   </link>
@@ -115,11 +154,24 @@
     </visual>
     <collision>
-      <geometry>
-        <cylinder radius="${wheel_radius}" length="${wheel_thickness}"/>
-      </geometry>
-    </collision>
-    <inertial>
-      <mass value="${wheel_mass}"/>
-      <inertia ixx="0.1" ixy="0.0" iyy="0.1" iyz="0.0" izz="0.1" ixz="0.0"/>
+      <origin xyz="0 0 0" rpy="0 0 0"/>
+      <geometry>
+        <cylinder radius="${wheel_radius}" length="${wheel_thickness}"/>
+      </geometry>
+      <gazebo>
+        <mu1>0.6</mu1>
+        <mu2>0.55</mu2>
+        <kp>100000</kp>
+        <kd>500</kd>
+      </gazebo>
+    </collision>
+    <inertial>
+      <mass value="${wheel_mass}"/>
+      <inertia
+          ixx="${wheel_Ixx}"
+          ixy="0.0"
+          iyy="${wheel_Iyy}"
+          izz="${wheel_Izz}"
+          iyz="0.0"
+          ixz="0.0"/>
     </inertial>
   </link>
@@ -129,6 +181,7 @@
     <parent link="chassis"/>
     <child link="wheel_1"/>
-    <limit lower="-3.14" upper="3.14" effort="10" velocity="10"/>
-    <axis xyz="0 0 1"/>
+    <limit lower="-3.14" upper="3.14" effort="2" velocity="4"/>
+    <dynamics damping="0.2"/>
+    <axis xyz="0 0 -1"/>
   </joint>
   <joint name="second_wheel_joint" type="revolute">
@@ -136,6 +189,7 @@
     <parent link="chassis"/>
     <child link="wheel_2"/>
-    <limit lower="-3.14" upper="3.14" effort="10" velocity="10"/>
-    <axis xyz="0 0 1"/>
+    <limit lower="-3.14" upper="3.14" effort="2" velocity="4"/>
+    <dynamics damping="0.2"/>
+    <axis xyz="0 0 -1"/>
   </joint>
   <joint name="third_wheel_joint" type="revolute">
@@ -143,5 +197,6 @@
     <parent link="chassis"/>
     <child link="wheel_3"/>
-    <limit lower="-3.14" upper="3.14" effort="10" velocity="10"/>
+    <limit lower="-3.14" upper="3.14" effort="2" velocity="4"/>
+    <dynamics damping="0.2"/>
     <axis xyz="0 0 1"/>
   </joint>
@@ -150,8 +205,9 @@
     <parent link="chassis"/>
     <child link="wheel_4"/>
-    <limit lower="-3.14" upper="3.14" effort="10" velocity="10"/>
+    <limit lower="-3.14" upper="3.14" effort="2" velocity="4"/>
+    <dynamics damping="0.2"/>
     <axis xyz="0 0 1"/>
   </joint>
-  <!-- ros2_control configuration using velocity command interfaces for each wheel -->
+  <!-- ros2_control configuration -->
   <ros2_control name="Gazebosim" type="system">
     <hardware>
@@ -179,9 +235,9 @@
     </joint>
   </ros2_control>
-  <!-- Gazebo plugin for ros2_control -->
   <gazebo>
     <plugin name="gazebo_ros2_control" filename="libgazebo_ros2_control.so">
-      <robotNamespace>/</robotNamespace>
+      <robot_namespace>/</robot_namespace>
       <parameters>$(find four_wheel_mobile_robot_navigation)/config/my_controllers.yaml</parameters>
+      <controller_manager_node_name>controller_manager</controller_manager_node_name>
     </plugin>
   </gazebo>
